Commit message: added collision and inertia to all parts

File: urdf/mobile_base.xacro (robot description, xacro)
@@ -74,4 +74,12 @@
             <material name="gray"/>
         </visual>
+        <collision>
+            <geometry>
+                <cylinder radius="${second_link_radius}" length="${second_link_height}"/>
+            </geometry>
+            <origin xyz="0 0 ${second_link_height/2.0}" rpy="0 0 0"/>
+        </collision>
+        <xacro:cylinder_inertia m="0.1" r="${second_link_radius}" l="${second_link_height}"
+                                xyz="0 0 ${second_link_height/2.0}" rpy="0 0 0"/>
     </link>
     <link name="third_link">
@@ -83,4 +91,12 @@
             <material name="red"/>
         </visual>
+        <collision>
+            <geometry>
+                <box size="${box_length} ${box_length} ${box_length}" />
+            </geometry>
+            <origin xyz="0 0 ${box_length/2.0}" rpy="0 0 0" />
+        </collision>
+        <xacro:box_inertia m="0.1" l="${box_length}" w="${box_length}" h="${box_length}"
+                           xyz="0 0 ${box_length/2.0}" rpy="0 0 0"/>
     </link>
     <link name="base_footprint_link">

Commit message: added camera and open CV orientation fix

File: urdf/mobile_base.xacro (robot description, xacro)
@@ -112,7 +112,7 @@
         <origin xyz="0 0 ${base_height}" rpy="0 0 0"/>
         <axis xyz="1 0 0" />
-        <limit lower="-0.3" upper="0.3" velocity="100" effort="100"/>
+        <limit lower="-0.18" upper="0.18" velocity="100" effort="100"/>
     </joint>
-    <joint name="secon_to_third_link_joint" type="revolute">
+    <joint name="second_to_third_link_joint" type="revolute">
         <parent link="second_link"/>
         <child link="third_link"/>

File: urdf/my_robot.urdf.xacro (robot description, xacro)
@@ -4,3 +4,4 @@
     <xacro:include filename="mobile_base.xacro"/>
     <xacro:include filename="mobile_base_gazebo.xacro"/>
+    <xacro:include filename="camera.xacro"/>
 </robot>

Commit message: standalone arm integration

File: urdf/mobile_base.xacro (robot description, xacro)
@@ -138,3 +138,9 @@
         <origin xyz="${base_length/3.0} 0 0" rpy="0 0 0"/>
     </joint>
+    <joint name="base_to_arm_base_joint" type="fixed">
+        <parent link="base_link"/>
+        <child link="arm_base_link"/>
+        <origin xyz="0 0 0" rpy="0 0 0"/>
+        <axis xyz="0 0 0" />
+    </joint>
 </robot>

File: urdf/my_robot.urdf.xacro (robot description, xacro)
@@ -5,3 +5,4 @@
     <xacro:include filename="mobile_base_gazebo.xacro"/>
     <xacro:include filename="camera.xacro"/>
+    <xacro:include filename="arm.xacro"/>
 </robot>
