Commit message: arm added

File: urdf/arm.xacro (robot description, xacro)
@@ -21,5 +21,5 @@
             <origin xyz="0 0 ${arm_base_heigth/2.0}" rpy="0 0 0" />
         </collision>
-        <xacro:box_inertia m="0.5" l="${arm_base_length}" w="${arm_base_width}" h="${arm_base_heigth}"
+        <xacro:box_inertia m="0.5" l="${2*arm_base_length}" w="${2*arm_base_width}" h="${2*arm_base_heigth}"
                            xyz="0 0 ${arm_base_heigth/2.0}" rpy="0 0 0"/>
     </link>
@@ -37,5 +37,5 @@
             <origin xyz="0 0 ${forearm_length/2.0}" rpy="0 0 0" />
         </collision>
-        <xacro:cylinder_inertia m="0.3" r="${forearm_radius}" l="${forearm_length}"
+        <xacro:cylinder_inertia m="0.4" r="${forearm_radius}" l="${forearm_length}"
                                     xyz="0 0 0" rpy="0 0 0"/>
     </link>
@@ -53,5 +53,5 @@
             <origin xyz="0 0 ${hand_length/2.0}" rpy="0 0 0" />
         </collision>
-        <xacro:cylinder_inertia m="0.3" r="${hand_radius}" l="${hand_length}"
+        <xacro:cylinder_inertia m="0.4" r="${hand_radius}" l="${hand_length}"
                                     xyz="0 0 0" rpy="0 0 0"/>
     </link>
@@ -62,5 +62,5 @@
         <axis xyz="0 1 0"/>
         <limit lower="0" upper="${pi/2.0}" velocity="100" effort="100"/>
-        <dynamics friction="0.05" damping="0.1"/>
+        <dynamics friction="0.01" damping="0.01"/>
     </joint>
     <joint name="forearm_hand_joint" type="revolute">
@@ -70,5 +70,5 @@
         <axis xyz="0 1 0" />
         <limit lower="0" upper="${pi/2.0}" velocity="100" effort="100"/>
-        <dynamics friction="0.05" damping="0.1"/>
+        <dynamics friction="0.01" damping="0.01"/>
     </joint>
 </robot>

File: urdf/mobile_base.xacro (robot description, xacro)
@@ -26,5 +26,5 @@
             <origin xyz="0 0 ${base_height/2.0}" rpy="0 0 0" />
         </collision>
-        <xacro:box_inertia m="${box_mass}" l="${base_length}" w="${base_width}" h="${base_height}"
+        <xacro:box_inertia m="${box_mass}" l="${2*base_length}" w="${2*base_width}" h="${2*base_height}"
                            xyz="0 0 ${base_height/2.0}" rpy="0 0 0"/>
     </link>
@@ -112,5 +112,5 @@
         <origin xyz="0 0 ${base_height}" rpy="0 0 0"/>
         <axis xyz="1 0 0" />
-        <limit lower="-0.18" upper="0.18" velocity="100" effort="100"/>
+        <limit lower="-0.1" upper="0.1" velocity="100" effort="100"/>
     </joint>
     <joint name="second_to_third_link_joint" type="revolute">
@@ -138,9 +138,3 @@
         <origin xyz="${base_length/3.0} 0 0" rpy="0 0 0"/>
     </joint>
-    <joint name="base_to_arm_base_joint" type="fixed">
-        <parent link="base_link"/>
-        <child link="arm_base_link"/>
-        <origin xyz="0 0 0" rpy="0 0 0"/>
-        <axis xyz="0 0 0" />
-    </joint>
 </robot>

File: urdf/my_robot.urdf.xacro (robot description, xacro)
@@ -4,5 +4,11 @@
     <xacro:include filename="mobile_base.xacro"/>
     <xacro:include filename="mobile_base_gazebo.xacro"/>
-    <xacro:include filename="camera.xacro"/>
+    --<xacro:include filename="camera.xacro"/>
+    <xacro:include filename="arm_properties.xacro"/>
     <xacro:include filename="arm.xacro"/>
+    <joint name="base_arm_base_joint" type="fixed">
+        <parent link="base_link"/>
+        <child link="arm_base_link"/>
+        <origin xyz="${(base_length/2.0)-(0.1/2.0)} 0 ${base_height}" rpy="0 0 0"/>
+    </joint>
 </robot>
